File: ANALOG_VTX.kicad_sch (KiCad schematic)
At the start: 11 parts, among them U5 AT7456ELAH, Y2 XL7EL89COI-111YLC-27M

Commit message: fixed some BOM issues
Parts:
- C20, C21, C22, C25: MPN GRM022R60J104KE15D -> CL05B104KO5NNNC
Changed lines of the file:
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@@
 			)
 		)
-		(property "MPN" "GRM022R60J104KE15D"
+		(property "MPN" "CL05B104KO5NNNC"
 			(at 135.89 72.39 90)
 			(hide yes)
@@
 			)
 		)
-		(property "MPN" "GRM022R60J104KE15D"
+		(property "MPN" "CL05B104KO5NNNC"
 			(at 63.5 48.26 0)
 			(hide yes)
@@
 			)
 		)
-		(property "MPN" "GRM022R60J104KE15D"
+		(property "MPN" "CL05B104KO5NNNC"
 			(at 53.34 39.37 0)
 			(hide yes)
@@
 			)
 		)
-		(property "MPN" "GRM022R60J104KE15D"
+		(property "MPN" "CL05B104KO5NNNC"
 			(at 73.66 57.15 0)
 			(hide yes)
