File: GNSS.kicad_sch (KiCad schematic)
At the start: 10 parts, among them CN1 CONMHF4-SMD-G-T, U11 MAX-M10S

Commit message: fixed some BOM issues
Parts:
- C42, C43: MPN GRM022R60J104KE15D -> CL05B104KO5NNNC
- L1: value 27nH -> 2.7nH
Changed lines of the file:
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@@
 			)
 		)
-		(property "MPN" "GRM022R60J104KE15D"
+		(property "MPN" "CL05B104KO5NNNC"
 			(at 115.57 31.75 0)
 			(hide yes)
@@
 			)
 		)
-		(property "MPN" "GRM022R60J104KE15D"
+		(property "MPN" "CL05B104KO5NNNC"
 			(at 106.68 31.75 0)
 			(hide yes)
@@
 			)
 		)
-		(property "Value" "27nH"
+		(property "Value" "2.7nH"
 			(at 133.35 49.53 90)
 			(show_name no)
