File: MCU.kicad_sch (KiCad schematic)
At the start: 35 parts, among them Q1 AO3400A, SW1 RKCGG140SMTRLFS, U1 STM32H743VIHx, U2 ZX-SH1.0-4PWT, Y1 8MHz

Commit message: fixed some BOM issues
Parts:
- C12, C13, C3, C7, C8, C9: MPN GRM022R60J104KE15D -> CL05B104KO5NNNC
