File: MICRO_SD.kicad_sch (KiCad schematic)
At the start: 9 parts, among them J1 TF-028-H265

Commit message: fixed some BOM issues
Parts:
- C40: MPN GRM022R60J104KE15D -> CL05B104KO5NNNC
Changed lines of the file:
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@@
 			)
 		)
-		(property "MPN" "GRM022R60J104KE15D"
+		(property "MPN" "CL05B104KO5NNNC"
 			(at 59.69 62.23 0)
 			(hide yes)
